File: pcb/board.kicad_sch (KiCad schematic)
At the start: 2 parts

Commit message: 2 led
Parts:
- added D2: LED_Small, LED_SMD:LED_0805_2012Metric, symbol Device:LED_Small
- added R2: R_Small, Resistor_SMD:R_0805_2012Metric, symbol Device:R_Small
Connections:
- net +3V3: now also R2.1
- net GND: now also D2.1 (K)
- new net: D2.2 (A), R2.2
